File: umod4.brd (EAGLE design)
At the start: 104.9 x 69.8 mm, 101 parts, among them IC1 27C256-FEED-THRU, M1 Generic single-sided NEO-8, M2 RPi Pico W, Q1 DNP/SI2301CDS, Q2 SS8050, U1 RP2040, U2 W25Q128JVSIQ, U3 SY6280AAC, U4 74LVC2G04, U5 74LVC541, U6 74LVC541, U7 74LVC4245, U8 TLV75733P, Y1 12MHz

Commit message: Replace 1K 0402 packages with SMD-0603-NOM
- Affected parts: R6, R10, R14, R27
- LCSC_PART changes from C11702 to C21190
- Manually reworked wire angles on board to clear DRC failures from the new pad geometry
Parts:
- R10, R14, R27, R6: device SparkFun-03-01-2010:0402-RES -> robins-v7:SMD-0603-NOM
- moved R10 0.25 mm to (87.9, 35.6)
Routing:
- net GND: track 5.09 -> 5.61 mm
Changed lines of the file:
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@@
 </element>
 <element name="C14" library="SparkFun-03-01-2010" package="0402-CAP" value="100n/16V/X7R" x="89.662" y="35.814" smashed="yes" rot="R270">
-<attribute name="NAME" x="88.8365" y="34.417" size="0.8128" layer="25" font="vector" ratio="14" rot="R270"/>
+<attribute name="NAME" x="89.0905" y="34.417" size="0.8128" layer="25" font="vector" ratio="14" rot="R270"/>
 <attribute name="VALUE" x="88.519" y="36.8935" size="0.4064" layer="27" rot="R270"/>
 <attribute name="LCSC_PART" value="C1525" x="89.662" y="35.814" size="1.778" layer="27" rot="R270" display="off"/>
@@
 <attribute name="LCSC_PART" value="C9002" x="85.09" y="33.782" size="1.778" layer="27" rot="R90" display="off"/>
 </element>
-<element name="R10" library="SparkFun-03-01-2010" package="0402-RES" value="1K" x="87.884" y="35.814" smashed="yes" rot="R270">
-<attribute name="NAME" x="88.2015" y="37.211" size="0.8128" layer="25" font="vector" ratio="14" rot="R90"/>
-<attribute name="VALUE" x="86.741" y="36.8935" size="0.4064" layer="27" rot="R270"/>
-<attribute name="LCSC_PART" value="C11702" x="87.884" y="35.814" size="1.778" layer="27" rot="R270" display="off"/>
+<element name="R10" library="robins-v7" package="SMD-0603-NOM" value="1K" x="87.884" y="35.56" smashed="yes" rot="R270">
+<attribute name="NAME" x="88.2015" y="36.957" size="0.8128" layer="25" font="vector" ratio="14" rot="R90"/>
+<attribute name="VALUE" x="86.741" y="36.6395" size="0.4064" layer="27" rot="R270"/>
+<attribute name="LCSC_PART" value="C21190" x="87.884" y="35.56" size="1.778" layer="27" rot="R270" display="off"/>
 </element>
 <element name="C11" library="SparkFun-03-01-2010" package="0402-CAP" value="33p/6.3V/COG" x="85.09" y="36.83" smashed="yes">
@@
 <attribute name="VALUE" x="76.994" y="5.818" size="1.27" layer="27" rot="R270"/>
 </element>
-<element name="R27" library="SparkFun-03-01-2010" package="0402-RES" value="1K" x="76.962" y="3.81" smashed="yes" rot="R90">
-<attribute name="LCSC_PART" value="C11702" x="76.962" y="3.81" size="1.778" layer="27" rot="R90" display="off"/>
+<element name="R27" library="robins-v7" package="SMD-0603-NOM" value="1K" x="76.962" y="3.81" smashed="yes" rot="R90">
+<attribute name="LCSC_PART" value="C21190" x="76.962" y="3.81" size="1.778" layer="27" rot="R90" display="off"/>
 <attribute name="NAME" x="78.105" y="2.3495" size="0.8128" layer="25" font="vector" ratio="14" rot="R180"/>
 <attribute name="VALUE" x="78.105" y="2.7305" size="0.4064" layer="27" rot="R90"/>
@@
 <attribute name="VALUE" x="5.056" y="13.684" size="1.27" layer="27" rot="R180"/>
 </element>
-<element name="R6" library="SparkFun-03-01-2010" package="0402-RES" value="1K" x="59.69" y="40.64" smashed="yes" rot="R90">
-<attribute name="LCSC_PART" value="C11702" x="59.69" y="40.64" size="1.778" layer="27" rot="R90" display="off"/>
+<element name="R6" library="robins-v7" package="SMD-0603-NOM" value="1K" x="59.69" y="40.64" smashed="yes" rot="R90">
+<attribute name="LCSC_PART" value="C21190" x="59.69" y="40.64" size="1.778" layer="27" rot="R90" display="off"/>
 <attribute name="NAME" x="60.2615" y="42.291" size="0.8128" layer="25" font="vector" ratio="14" rot="R90"/>
 <attribute name="VALUE" x="60.833" y="39.5605" size="0.4064" layer="27" rot="R90"/>
@@
 <attribute name="VALUE" x="64.0715" y="19.431" size="0.4064" layer="27" rot="R180"/>
 </element>
-<element name="R14" library="SparkFun-03-01-2010" package="0402-RES" value="1K" x="66.294" y="33.02" smashed="yes" rot="R90">
-<attribute name="LCSC_PART" value="C11702" x="66.294" y="33.02" size="0.8128" layer="27" ratio="14" rot="R90" display="off"/>
+<element name="R14" library="robins-v7" package="SMD-0603-NOM" value="1K" x="66.294" y="33.02" smashed="yes" rot="R90">
+<attribute name="LCSC_PART" value="C21190" x="66.294" y="33.02" size="0.8128" layer="27" ratio="14" rot="R90" display="off"/>
 <attribute name="NAME" x="67.2465" y="34.163" size="0.8128" layer="25" font="vector" ratio="14" rot="R270"/>
 <attribute name="VALUE" x="67.437" y="31.9405" size="0.4064" layer="27" rot="R90"/>
@@
 <contactref element="C1" pad="2"/>
 <contactref element="Q2" pad="2"/>
-<wire x1="83.332" y1="32.584" x2="83.932" y2="32.584" width="0.2032" layer="1"/>
-<wire x1="85.946" y1="36.092" x2="85.946" y2="35.438" width="0.2032" layer="1"/>
 <contactref element="R18" pad="2"/>
 <contactref element="JP2" pad="2"/>
@@
 <contactref element="C17" pad="2"/>
 <contactref element="TP16" pad="P$1"/>
+<wire x1="84.328" y1="32.512" x2="83.312" y2="32.512" width="0.254" layer="1"/>
+<wire x1="85.852" y1="34.798" x2="85.852" y2="34.036" width="0.254" layer="1"/>
 </signal>
 <signal name="+3V3">
@@
 <wire x1="4.127" y1="13.716" x2="4.127" y2="14.161" width="0.3048" layer="1"/>
 <wire x1="4.127" y1="14.161" x2="3.556" y2="14.732" width="0.3048" layer="1"/>
-<wire x1="90.932" y1="46.228" x2="91.5247" y2="45.9324" width="0" layer="19" extent="1-1"/>
-<wire x1="90.6872" y1="46.7699" x2="90.932" y2="46.228" width="0" layer="19" extent="1-1"/>
-<wire x1="90.2872" y1="46.7699" x2="90.6872" y2="46.7699" width="0" layer="19" extent="1-1"/>
-<wire x1="88.6872" y1="46.7699" x2="90.2872" y2="46.7699" width="0" layer="19" extent="1-1"/>
-<wire x1="85.852" y1="45.72" x2="88.2872" y2="46.7699" width="0" layer="19" extent="1-16"/>
-<wire x1="83.0844" y1="42.3324" x2="83.312" y2="43.18" width="0" layer="19" extent="1-16"/>
-<wire x1="84.6497" y1="45.9324" x2="85.344" y2="45.212" width="0" layer="19" extent="1-16"/>
-<wire x1="91.5247" y1="42.3324" x2="91.5247" y2="45.9324" width="0" layer="19" extent="1-1"/>
-<wire x1="88.2872" y1="39.8949" x2="91.5247" y2="42.3324" width="0" layer="19" extent="1-1"/>
 <wire x1="101.854" y1="6.795" x2="101.805" y2="6.795" width="0.3048" layer="1"/>
 <wire x1="101.805" y1="6.795" x2="101.742" y2="6.858" width="0.3048" layer="1"/>
@@
 <contactref element="R10" pad="2"/>
 <contactref element="C18" pad="2"/>
-<wire x1="87.884" y1="33.416" x2="87.884" y2="35.164" width="0.2032" layer="1"/>
+<wire x1="87.884" y1="33.416" x2="87.884" y2="34.735" width="0.2032" layer="1"/>
 <wire x1="87.884" y1="33.416" x2="86.774" y2="33.416" width="0.2032" layer="1"/>
 <wire x1="86.774" y1="33.416" x2="85.965" y2="32.607" width="0.2032" layer="1"/>
@@
 <contactref element="R10" pad="1"/>
 <wire x1="87.8872" y1="39.8949" x2="87.8872" y2="36.4672" width="0.2032" layer="1"/>
-<wire x1="87.8872" y1="36.4672" x2="87.884" y2="36.464" width="0.2032" layer="1"/>
+<wire x1="87.8872" y1="36.4672" x2="87.8872" y2="36.3882" width="0.254" layer="1"/>
+<wire x1="87.8872" y1="36.3882" x2="87.884" y2="36.385" width="0.254" layer="1"/>
 </signal>
 <signal name="N$6">
@@
 <wire x1="67.2592" y1="37.211" x2="66.167" y2="37.211" width="0.2032" layer="1"/>
 <contactref element="R6" pad="1"/>
-<wire x1="61.468" y1="39.99" x2="59.69" y2="39.99" width="0.3048" layer="1"/>
 <contactref element="R14" pad="2"/>
-<wire x1="66.294" y1="33.67" x2="66.294" y2="35.306" width="0.254" layer="1"/>
+<wire x1="66.294" y1="33.845" x2="66.294" y2="35.306" width="0.254" layer="1"/>
 <wire x1="66.294" y1="35.306" x2="66.548" y2="35.56" width="0.254" layer="1"/>
 <wire x1="66.548" y1="35.56" x2="67.437" y2="35.56" width="0.254" layer="1"/>
+<wire x1="61.468" y1="39.99" x2="59.69" y2="39.99" width="0.3048" layer="1"/>
+<wire x1="59.69" y1="39.99" x2="59.69" y2="39.815" width="0.3048" layer="1"/>
 </signal>
 <signal name="N$9">
@@
 <wire x1="79.8572" y1="25.257" x2="79.8572" y2="24.2828" width="0.4064" layer="1"/>
 <wire x1="79.8572" y1="24.2828" x2="80.01" y2="24.13" width="0.4064" layer="1"/>
-<wire x1="76.962" y1="3.16" x2="76.962" y2="2.794" width="0.254" layer="1"/>
-<wire x1="76.962" y1="2.794" x2="76.2" y2="2.032" width="0.3048" layer="1"/>
-<wire x1="76.2" y1="2.032" x2="56.896" y2="2.032" width="0.3048" layer="1"/>
+<wire x1="76.962" y1="2.985" x2="76.962" y2="2.794" width="0.254" layer="1"/>
+<wire x1="76.708" y1="2.032" x2="56.896" y2="2.032" width="0.3048" layer="1"/>
 <via x="56.388" y="2.54" extent="1-16" drill="0.7112"/>
 <wire x1="56.388" y1="2.54" x2="55.88" y2="2.032" width="0.3048" layer="16"/>
@@
 <wire x1="57.404" y1="3.556" x2="57.404" y2="10.922" width="0.3048" layer="1"/>
 <wire x1="57.404" y1="10.922" x2="59.944" y2="13.462" width="0.3048" layer="1"/>
+<wire x1="76.962" y1="2.794" x2="76.962" y2="2.286" width="0.3048" layer="1"/>
+<wire x1="76.962" y1="2.286" x2="76.708" y2="2.032" width="0.3048" layer="1"/>
 </signal>
 <signal name="N$3">
@@
 <wire x1="78.994" y1="3.268" x2="78.774" y2="3.268" width="0.254" layer="1"/>
 <wire x1="78.774" y1="3.268" x2="77.582" y2="4.46" width="0.254" layer="1"/>
-<wire x1="76.962" y1="4.46" x2="77.582" y2="4.46" width="0.254" layer="1"/>
+<wire x1="76.962" y1="4.635" x2="77.407" y2="4.635" width="0.254" layer="1"/>
+<wire x1="77.407" y1="4.635" x2="77.582" y2="4.46" width="0.254" layer="1"/>
 </signal>
 <signal name="N$19">
@@
 <contactref element="M2" pad="27"/>
 <contactref element="R6" pad="2"/>
-<wire x1="59.69" y1="41.29" x2="54.498" y2="41.29" width="0.3048" layer="1"/>
 <wire x1="54.498" y1="41.29" x2="54.356" y2="41.148" width="0.3048" layer="1"/>
 <via x="54.356" y="41.148" extent="1-16" drill="0.508"/>
@@
 <wire x1="37.338" y1="24.638" x2="28.448" y2="15.748" width="0.3048" layer="1"/>
 <wire x1="28.448" y1="15.748" x2="28.448" y2="8.128" width="0.3048" layer="1"/>
+<wire x1="59.69" y1="41.465" x2="54.356" y2="41.465" width="0.3048" layer="1"/>
+<wire x1="54.356" y1="41.465" x2="54.356" y2="41.148" width="0.3048" layer="1"/>
 </signal>
 <signal name="SPARE0_ADC">
@@
 <wire x1="64.262" y1="30.734" x2="65.532" y2="30.734" width="0.3048" layer="1"/>
 <wire x1="65.532" y1="30.734" x2="66.294" y2="31.496" width="0.3048" layer="1"/>
-<wire x1="66.294" y1="31.496" x2="66.294" y2="32.37" width="0.3048" layer="1"/>
+<wire x1="66.294" y1="31.496" x2="66.294" y2="32.195" width="0.3048" layer="1"/>
 </signal>
 <signal name="SPARE6_ADC">

Commit message: Replace 4K7 0603 packages with SMD-0603-NOM
- Affected parts: R4
- LCSC_PART is unchanged
- Manually reworked wire angles on board to clear DRC failures from the new pad geometry
Parts:
- R4: device SparkFun-03-01-2010:0603-RES -> robins-v7:SMD-0603-NOM
Changed lines of the file:
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@@
 <attribute name="VALUE" x="90.3605" y="53.975" size="0.4064" layer="27"/>
 </element>
-<element name="R4" library="SparkFun-03-01-2010" package="0603-RES" value="4K7" x="95.758" y="55.118" smashed="yes" rot="R180">
+<element name="R4" library="robins-v7" package="SMD-0603-NOM" value="4K7" x="95.758" y="55.118" smashed="yes" rot="R180">
 <attribute name="NAME" x="97.663" y="54.8005" size="0.8128" layer="25" font="vector" ratio="14"/>
 <attribute name="VALUE" x="96.8375" y="56.261" size="0.4064" layer="27" rot="R180"/>
@@
 <contactref element="R4" pad="1"/>
 <wire x1="93.33" y1="49.276" x2="93.33" y2="50.404" width="0.3048" layer="1"/>
-<wire x1="93.33" y1="50.404" x2="96.608" y2="53.682" width="0.3048" layer="1"/>
+<wire x1="93.33" y1="50.404" x2="96.583" y2="53.657" width="0.3048" layer="1"/>
 <wire x1="49.022" y1="30.368" x2="51.166" y2="30.368" width="0.3048" layer="1"/>
 <wire x1="51.166" y1="30.368" x2="51.308" y2="30.226" width="0.3048" layer="1"/>
@@
 <wire x1="88.6872" y1="47.7932" x2="88.2872" y2="47.3932" width="0.254" layer="1"/>
 <wire x1="88.2872" y1="46.7699" x2="88.2872" y2="47.3932" width="0.254" layer="1"/>
-<wire x1="96.608" y1="55.118" x2="96.608" y2="53.682" width="0.3048" layer="1"/>
 <wire x1="51.45" y1="35.194" x2="51.308" y2="35.052" width="0.2032" layer="1"/>
 <wire x1="51.45" y1="35.194" x2="54.102" y2="35.194" width="0.3048" layer="1"/>
@@
 <wire x1="101.854" y1="6.795" x2="101.805" y2="6.795" width="0.3048" layer="1"/>
 <wire x1="101.805" y1="6.795" x2="101.742" y2="6.858" width="0.3048" layer="1"/>
+<wire x1="96.583" y1="55.118" x2="96.583" y2="53.657" width="0.3048" layer="1"/>
 </signal>
 <signal name="R/!W!_5V">
@@
 <wire x1="94.996" y1="57.912" x2="94.996" y2="56.134" width="0.3048" layer="1"/>
 <wire x1="94.996" y1="56.134" x2="94.996" y2="55.206" width="0.3048" layer="1"/>
-<wire x1="94.996" y1="55.206" x2="94.908" y2="55.118" width="0.3048" layer="1"/>
+<wire x1="94.933" y1="55.118" x2="94.933" y2="55.143" width="0.3048" layer="1"/>
+<wire x1="94.933" y1="55.143" x2="94.996" y2="55.206" width="0.3048" layer="1"/>
 </signal>
 <signal name="IO0">

Commit message: Replace 100R 0603 packages with SMD-0603-NOM
- Affected parts: R1, R2, R20
- LCSC_PART unchanged
- Manually reworked wire angles on board to clear DRC failures from the new pad geometry
Parts:
- R1, R2, R20: device SparkFun-03-01-2010:0603-RES -> robins-v7:SMD-0603-NOM
Changed lines of the file:
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@@
 <attribute name="VALUE" x="44.577" y="34.29" size="1.27" layer="27" rot="R90"/>
 </element>
-<element name="R20" library="SparkFun-03-01-2010" package="0603-RES" value="100R" x="87.63" y="27.178" smashed="yes" rot="R270">
+<element name="R20" library="robins-v7" package="SMD-0603-NOM" value="100R" x="87.63" y="27.178" smashed="yes" rot="R270">
 <attribute name="LCSC_PART" value="C22775" x="87.63" y="27.178" size="1.778" layer="27" ratio="14" rot="R270" display="off"/>
-<attribute name="NAME" x="88.5825" y="28.829" size="0.8128" layer="25" ratio="14" rot="R270"/>
+<attribute name="NAME" x="88.5825" y="28.321" size="0.8128" layer="25" ratio="14" rot="R270"/>
 <attribute name="VALUE" x="86.487" y="28.2575" size="0.4064" layer="27" rot="R270"/>
 </element>
@@
 <attribute name="VALUE" x="78.105" y="2.7305" size="0.4064" layer="27" rot="R90"/>
 </element>
-<element name="R1" library="SparkFun-03-01-2010" package="0603-RES" value="100R" x="91.44" y="57.912" smashed="yes">
+<element name="R1" library="robins-v7" package="SMD-0603-NOM" value="100R" x="91.44" y="57.912" smashed="yes">
 <attribute name="NAME" x="89.789" y="58.4835" size="0.8128" layer="25" ratio="14" rot="R180"/>
 <attribute name="VALUE" x="90.3605" y="56.769" size="0.4064" layer="27"/>
 <attribute name="LCSC_PART" value="C22775" x="91.44" y="57.912" size="1.778" layer="27" display="off"/>
 </element>
-<element name="R2" library="SparkFun-03-01-2010" package="0603-RES" value="100R" x="95.758" y="57.912" smashed="yes">
+<element name="R2" library="robins-v7" package="SMD-0603-NOM" value="100R" x="95.758" y="57.912" smashed="yes">
 <attribute name="NAME" x="97.663" y="57.5945" size="0.8128" layer="25" ratio="14"/>
 <attribute name="VALUE" x="94.6785" y="56.769" size="0.4064" layer="27"/>
@@
 <wire x1="85.964" y1="28.336" x2="85.852" y2="28.448" width="0.2032" layer="1"/>
 <wire x1="85.652" y1="28.648" x2="85.852" y2="28.448" width="0.2032" layer="1"/>
-<wire x1="87.63" y1="28.028" x2="86.272" y2="28.028" width="0.2032" layer="1"/>
-<wire x1="86.272" y1="28.028" x2="85.852" y2="28.448" width="0.2032" layer="1"/>
+<wire x1="86.297" y1="28.003" x2="85.852" y2="28.448" width="0.2032" layer="1"/>
+<wire x1="87.63" y1="28.003" x2="86.297" y2="28.003" width="0.2032" layer="1"/>
 </signal>
 <signal name="RP_SWCLK">
@@
 <wire x1="89.662" y1="56.896" x2="89.408" y2="56.642" width="0.2032" layer="16"/>
 <wire x1="90.79" y1="56.642" x2="90.79" y2="57.712" width="0.3048" layer="1"/>
-<wire x1="90.79" y1="57.712" x2="90.59" y2="57.912" width="0.3048" layer="1"/>
 <wire x1="50.038" y1="25.4" x2="50.8" y2="24.638" width="0.2032" layer="16"/>
 <wire x1="50.8" y1="24.638" x2="52.578" y2="24.638" width="0.2032" layer="16"/>
 <wire x1="52.578" y1="24.638" x2="53.848" y2="25.908" width="0.2032" layer="16"/>
+<wire x1="90.615" y1="57.912" x2="90.79" y2="57.912" width="0.4064" layer="1"/>
+<wire x1="90.79" y1="57.912" x2="90.79" y2="57.712" width="0.4064" layer="1"/>
 </signal>
 <signal name="RP_SWD">
@@
 <via x="93.726" y="56.134" extent="1-16" drill="0.508"/>
 <wire x1="93.726" y1="56.134" x2="94.996" y2="56.134" width="0.3048" layer="1"/>
-<wire x1="94.908" y1="57.912" x2="94.996" y2="57.912" width="0.2032" layer="1"/>
+<wire x1="94.933" y1="57.912" x2="94.996" y2="57.912" width="0.2032" layer="1"/>
 <wire x1="94.996" y1="57.912" x2="94.996" y2="56.134" width="0.3048" layer="1"/>
 <wire x1="94.996" y1="56.134" x2="94.996" y2="55.206" width="0.3048" layer="1"/>
@@
 <contactref element="U6" pad="11"/>
 <wire x1="85.8008" y1="25.257" x2="85.8008" y2="26.1108" width="0.2032" layer="1"/>
-<wire x1="87.63" y1="26.328" x2="86.018" y2="26.328" width="0.2032" layer="1"/>
-<wire x1="86.018" y1="26.328" x2="85.8008" y2="26.1108" width="0.2032" layer="1"/>
+<wire x1="86.043" y1="26.353" x2="85.8008" y2="26.1108" width="0.2032" layer="1"/>
+<wire x1="87.63" y1="26.353" x2="86.043" y2="26.353" width="0.2032" layer="1"/>
 </signal>
 <signal name="WP_RUN">
@@
 <contactref element="JP1" pad="1"/>
 <contactref element="R1" pad="2"/>
-<wire x1="92.29" y1="59.348" x2="91.186" y2="60.452" width="0.4064" layer="1"/>
-<wire x1="91.186" y1="60.452" x2="91.186" y2="62.992" width="0.4064" layer="1"/>
-<wire x1="92.29" y1="57.912" x2="92.29" y2="59.348" width="0.4064" layer="1"/>
+<wire x1="91.186" y1="60.198" x2="91.186" y2="62.992" width="0.4064" layer="1"/>
+<wire x1="91.186" y1="60.198" x2="92.265" y2="59.119" width="0.4064" layer="1"/>
+<wire x1="92.265" y1="57.912" x2="92.265" y2="59.119" width="0.4064" layer="1"/>
 </signal>
 <signal name="EXT_RP_SWD">
@@
 <contactref element="R2" pad="2"/>
 <wire x1="96.266" y1="62.992" x2="96.266" y2="59.832" width="0.4064" layer="1"/>
-<wire x1="96.608" y1="57.912" x2="96.52" y2="57.912" width="0.4064" layer="1"/>
+<wire x1="96.583" y1="57.912" x2="96.52" y2="57.912" width="0.4064" layer="1"/>
 <wire x1="96.52" y1="57.912" x2="96.52" y2="59.578" width="0.4064" layer="1"/>
 <wire x1="96.52" y1="59.578" x2="96.266" y2="59.832" width="0.4064" layer="1"/>

Commit message: Replace 10K 0402 packages with SMD-0603-NOM
- Affected parts: R3, R5, R7, R8. R9, R11, R12, R13, R15, R16, R17, R18, R19, R22, R25, R26
- LCSC_PART changed to C25804 (10K 0603 1% basic)
- Manually reworked wire angles on board to clear DRC failures from the new pad geometry
Parts:
- R11, R12, R13, R15, R16, R17, R18, R19, R22, R25, R26, R3, R5, R7, R8, R9: device SparkFun-03-01-2010:0402-RES -> robins-v7:SMD-0603-NOM
